File: LED-driver.sch (KiCad schematic (older format))
At the start: 34 parts, among them J1 Screw_Terminal_1x02, J2 PIC Kit3 header, J3 Screw_Terminal_1x02, J4 Screw_Terminal_1x02, J5 Screw_Terminal_1x02, J6 Screw_Terminal_1x03, Q1 Q_NMOS_DGS, Q2 Q_NMOS_DGS, Q3 Q_NMOS_DGS, U1 PIC12F1572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

Commit message: Fix schematic-PCB references and update GBR files.
Parts:
- JP1: value Jumper_NC_Small -> MCLR
- JP2: value Jumper_NO_Small -> RX
- JP3: value Jumper_NO_Small -> TX
- R4: renamed from 510R1; value R -> 510R
- R5: renamed from 510R2; value R -> 510R
- R6: renamed from 510R3; value R -> 510R
- R7: renamed from 10K1; value R -> 10K
- R8: renamed from 10K5; value R -> 10K
- R9: renamed from 10K6; value R -> 10K
Changed lines of the file:
@@
 P 4100 5000
 F 0 "JP1" H 4100 5080 50  0000 C CNN
-F 1 "Jumper_NC_Small" H 4110 4940 50  0001 C CNN
+F 1 "MCLR" H 4110 4940 50  0001 C CNN
 F 2 "Pin_Headers:Pin_Header_Straight_1x02" H 4100 5000 50  0001 C CNN
 F 3 "" H 4100 5000 50  0001 C CNN
@@
 MCLR
 $Comp
-L R 10K1
+L R R7
 U 1 1 598997EF
 P 4450 5000
-F 0 "10K1" V 4530 5000 50  0000 C CNN
-F 1 "R" V 4450 5000 50  0000 C CNN
+F 0 "R7" V 4530 5000 50  0000 C CNN
+F 1 "10K" V 4450 5000 50  0000 C CNN
 F 2 "Resistors_SMD:R_0805_HandSoldering" V 4380 5000 50  0001 C CNN
 F 3 "" H 4450 5000 50  0001 C CNN
@@
 $EndComp
 $Comp
-L R 510R3
+L R R6
 U 1 1 5989A1D3
 P 4950 6450
-F 0 "510R3" V 5030 6450 50  0000 C CNN
-F 1 "R" V 4950 6450 50  0000 C CNN
+F 0 "R6" V 4850 6450 50  0000 C CNN
+F 1 "510R" V 4950 6450 50  0000 C CNN
 F 2 "Resistors_SMD:R_0805_HandSoldering" V 4880 6450 50  0001 C CNN
 F 3 "" H 4950 6450 50  0001 C CNN
@@
 $EndComp
 $Comp
-L R 510R1
+L R R4
 U 1 1 5989B6D2
 P 2300 6450
-F 0 "510R1" V 2380 6450 50  0000 C CNN
-F 1 "R" V 2300 6450 50  0000 C CNN
+F 0 "R4" V 2380 6450 50  0000 C CNN
+F 1 "510R" V 2300 6450 50  0000 C CNN
 F 2 "Resistors_SMD:R_0805_HandSoldering" V 2230 6450 50  0001 C CNN
 F 3 "" H 2300 6450 50  0001 C CNN
@@
 P 8200 3600
 F 0 "JP2" H 8200 3680 50  0000 C CNN
-F 1 "Jumper_NO_Small" H 8210 3540 50  0001 C CNN
+F 1 "RX" H 8210 3540 50  0001 C CNN
 F 2 "Pin_Headers:Pin_Header_Straight_1x02" H 8200 3600 50  0001 C CNN
 F 3 "" H 8200 3600 50  0001 C CNN
@@
 $EndComp
 $Comp
-L R 510R2
+L R R5
 U 1 1 59960D2A
 P 4200 6450
-F 0 "510R2" V 4280 6450 50  0000 C CNN
-F 1 "R" V 4200 6450 50  0000 C CNN
+F 0 "R5" V 4280 6450 50  0000 C CNN
+F 1 "510R" V 4200 6450 50  0000 C CNN
 F 2 "Resistors_SMD:R_0805_HandSoldering" V 4130 6450 50  0001 C CNN
 F 3 "" H 4200 6450 50  0001 C CNN
@@
 P 6000 4100
 F 0 "JP3" H 6000 4180 50  0000 C CNN
-F 1 "Jumper_NO_Small" H 6010 4040 50  0001 C CNN
+F 1 "TX" H 6010 4040 50  0001 C CNN
 F 2 "Pin_Headers:Pin_Header_Straight_1x02" H 6000 4100 50  0001 C CNN
 F 3 "" H 6000 4100 50  0001 C CNN
@@
 UART_TX/DAT
 $Comp
-L R 10K6
+L R R9
 U 1 1 59962180
 P 6900 3550
-F 0 "10K6" V 6980 3550 50  0000 C CNN
-F 1 "R" V 6900 3550 50  0000 C CNN
+F 0 "R9" V 6980 3550 50  0000 C CNN
+F 1 "10K" V 6900 3550 50  0000 C CNN
 F 2 "Resistors_SMD:R_0805_HandSoldering" V 6830 3550 50  0001 C CNN
 F 3 "" H 6900 3550 50  0001 C CNN
@@
 $EndComp
 $Comp
-L R 10K5
+L R R8
 U 1 1 599625DA
 P 6350 4100
-F 0 "10K5" V 6430 4100 50  0000 C CNN
-F 1 "R" V 6350 4100 50  0000 C CNN
+F 0 "R8" V 6430 4100 50  0000 C CNN
+F 1 "10K" V 6350 4100 50  0000 C CNN
 F 2 "Resistors_SMD:R_0805_HandSoldering" V 6280 4100 50  0001 C CNN
 F 3 "" H 6350 4100 50  0001 C CNN

Commit message: Tweak resistor values.
Parts:
- R1, R2, R3: value R_Small -> 1.4K
- R4, R5, R6: value 510R -> 511
Connections:
- wire segments 97 -> 98
Changed lines of the file:
@@
 U 1 1 597F76C7
 P 5750 1800
-F 0 "R2" H 5780 1820 50  0000 L CNN
-F 1 "R_Small" V 5780 1760 50  0001 L CNN
+F 0 "R2" V 5850 1700 50  0000 L CNN
+F 1 "1.4K" V 5950 1700 50  0000 L CNN
 F 2 "Resistors_SMD:R_0805_HandSoldering" H 5750 1800 50  0001 C CNN
 F 3 "" H 5750 1800 50  0001 C CNN
@@
 L GND #PWR05
 U 1 1 597F7A89
-P 3650 2800
-F 0 "#PWR05" H 3650 2550 50  0001 C CNN
-F 1 "GND" H 3650 2650 50  0000 C CNN
-F 2 "" H 3650 2800 50  0001 C CNN
-F 3 "" H 3650 2800 50  0001 C CNN
-	1    3650 2800
-	0    1    1    0
+P 3450 2700
+F 0 "#PWR05" H 3450 2450 50  0001 C CNN
+F 1 "GND" H 3450 2550 50  0000 C CNN
+F 2 "" H 3450 2700 50  0001 C CNN
+F 3 "" H 3450 2700 50  0001 C CNN
+	1    3450 2700
+	-1   0    0    1
 $EndComp
 $Comp
@@
 F 3 "" H 3650 2700 50  0001 C CNN
 	1    3650 2700
-	0    -1   -1   0
+	1    0    0    -1
 $EndComp
 $Comp
@@
 U 1 1 597F7F33
 P 3550 1800
-F 0 "R1" H 3580 1820 50  0000 L CNN
-F 1 "R_Small" V 3580 1760 50  0001 L CNN
+F 0 "R1" V 3650 1700 50  0000 L CNN
+F 1 "1.4K" V 3750 1700 50  0000 L CNN
 F 2 "Resistors_SMD:R_0805_HandSoldering" H 3550 1800 50  0001 C CNN
 F 3 "" H 3550 1800 50  0001 C CNN
@@
 U 1 1 597F805D
 P 7950 1800
-F 0 "R3" H 7980 1820 50  0000 L CNN
-F 1 "R_Small" V 7980 1760 50  0001 L CNN
+F 0 "R3" V 8050 1700 50  0000 L CNN
+F 1 "1.4K" V 8150 1700 50  0000 L CNN
 F 2 "Resistors_SMD:R_0805_HandSoldering" H 7950 1800 50  0001 C CNN
 F 3 "" H 7950 1800 50  0001 C CNN
@@
 P 4950 6450
 F 0 "R6" V 4850 6450 50  0000 C CNN
-F 1 "510R" V 4950 6450 50  0000 C CNN
+F 1 "511" V 4950 6450 50  0000 C CNN
 F 2 "Resistors_SMD:R_0805_HandSoldering" V 4880 6450 50  0001 C CNN
 F 3 "" H 4950 6450 50  0001 C CNN
@@
 P 2300 6450
 F 0 "R4" V 2380 6450 50  0000 C CNN
-F 1 "510R" V 2300 6450 50  0000 C CNN
+F 1 "511" V 2300 6450 50  0000 C CNN
 F 2 "Resistors_SMD:R_0805_HandSoldering" V 2230 6450 50  0001 C CNN
 F 3 "" H 2300 6450 50  0001 C CNN
@@
 P 4200 6450
 F 0 "R5" V 4280 6450 50  0000 C CNN
-F 1 "510R" V 4200 6450 50  0000 C CNN
+F 1 "511" V 4200 6450 50  0000 C CNN
 F 2 "Resistors_SMD:R_0805_HandSoldering" V 4130 6450 50  0001 C CNN
 F 3 "" H 4200 6450 50  0001 C CNN
@@
 	3650 2700 3700 2700
 Wire Wire Line
-	3650 2800 3700 2800
-Wire Wire Line
 	3650 2900 3700 2900
 Wire Wire Line
@@
 Wire Wire Line
 	4950 7050 4950 7200
+Wire Wire Line
+	3700 2800 3450 2800
+Wire Wire Line
+	3450 2800 3450 2700
 $EndSCHEMATC

Commit message: Final tweaks.
Parts:
- 0.1uF1, 0.1uF2, 0.1uF3, 0.1uF4, 0.1uF5: value CP -> 0.1uF
- Q1, Q2: value Q_NMOS_DGS -> 2N7002
- Q3: value Q_NMOS_DGS -> BSS123
Changed lines of the file:
@@
 U 1 1 597F7517
 P 2200 5150
-F 0 "0.1uF3" H 2210 5220 50  0000 L CNN
-F 1 "CP" H 2210 5070 50  0000 L CNN
+F 0 "0.1uF3" H 2210 5220 50  0001 L CNN
+F 1 "0.1uF" H 2210 5070 50  0000 L CNN
 F 2 "Capacitors_SMD:C_0805_HandSoldering" H 2200 5150 50  0001 C CNN
 F 3 "" H 2200 5150 50  0001 C CNN
@@
 U 1 1 597F7B56
 P 1400 5150
-F 0 "0.1uF2" H 1410 5220 50  0000 L CNN
-F 1 "CP" H 1410 5070 50  0000 L CNN
+F 0 "0.1uF2" H 1410 5220 50  0001 L CNN
+F 1 "0.1uF" H 1410 5070 50  0000 L CNN
 F 2 "Capacitors_SMD:C_0805_HandSoldering" H 1400 5150 50  0001 C CNN
 F 3 "" H 1400 5150 50  0001 C CNN
@@
 U 1 1 597F7F27
 P 2650 5150
-F 0 "0.1uF1" H 2660 5220 50  0000 L CNN
-F 1 "CP" H 2660 5070 50  0000 L CNN
+F 0 "0.1uF1" H 2660 5220 50  0001 L CNN
+F 1 "0.1uF" H 2660 5070 50  0000 L CNN
 F 2 "Capacitors_SMD:C_0805_HandSoldering" H 2650 5150 50  0001 C CNN
 F 3 "" H 2650 5150 50  0001 C CNN
@@
 U 1 1 597F8051
 P 1800 5150
-F 0 "0.1uF4" H 1810 5220 50  0000 L CNN
-F 1 "CP" H 1810 5070 50  0000 L CNN
+F 0 "0.1uF4" H 1810 5220 50  0001 L CNN
+F 1 "0.1uF" H 1810 5070 50  0000 L CNN
 F 2 "Capacitors_SMD:C_0805_HandSoldering" H 1800 5150 50  0001 C CNN
 F 3 "" H 1800 5150 50  0001 C CNN
@@
 U 1 1 597F8745
 P 1050 5150
-F 0 "0.1uF5" H 1060 5220 50  0000 L CNN
-F 1 "CP" H 1060 5070 50  0000 L CNN
+F 0 "0.1uF5" H 1060 5220 50  0001 L CNN
+F 1 "0.1uF" H 1060 5070 50  0000 L CNN
 F 2 "Capacitors_SMD:C_0805_HandSoldering" H 1050 5150 50  0001 C CNN
 F 3 "" H 1050 5150 50  0001 C CNN
@@
 L +5V #PWR025
 U 1 1 5989A391
-P 4950 6200
-F 0 "#PWR025" H 4950 6050 50  0001 C CNN
-F 1 "+5V" H 4950 6340 50  0000 C CNN
-F 2 "" H 4950 6200 50  0001 C CNN
-F 3 "" H 4950 6200 50  0001 C CNN
-	1    4950 6200
+P 4950 6250
+F 0 "#PWR025" H 4950 6100 50  0001 C CNN
+F 1 "+5V" H 4950 6390 50  0000 C CNN
+F 2 "" H 4950 6250 50  0001 C CNN
+F 3 "" H 4950 6250 50  0001 C CNN
+	1    4950 6250
 	1    0    0    -1
 $EndComp
@@
 P 1800 6950
 F 0 "Q1" H 2000 6950 50  0000 L CNN
-F 1 "Q_NMOS_DGS" V 2000 6900 50  0001 L CNN
+F 1 "2N7002" H 2000 6850 50  0000 L CNN
 F 2 "TO_SOT_Packages_SMD:SOT-23_Handsoldering" H 2000 7050 50  0001 C CNN
 F 3 "" H 1800 6950 50  0001 C CNN
@@
 P 3700 6950
 F 0 "Q2" H 3900 6950 50  0000 L CNN
-F 1 "Q_NMOS_DGS" H 3900 6900 50  0001 L CNN
+F 1 "2N7002" H 3900 6850 50  0000 L CNN
 F 2 "TO_SOT_Packages_SMD:SOT-23_Handsoldering" H 3900 7050 50  0001 C CNN
 F 3 "" H 3700 6950 50  0001 C CNN
@@
 P 6800 4100
 F 0 "Q3" H 7000 4100 50  0000 L CNN
-F 1 "Q_NMOS_DGS" H 7000 4050 50  0001 L CNN
+F 1 "BSS123" H 7000 4000 50  0000 L CNN
 F 2 "TO_SOT_Packages_SMD:SOT-23_Handsoldering" H 7000 4200 50  0001 C CNN
 F 3 "" H 6800 4100 50  0001 C CNN
@@
 	1400 3800 1400 3900
 Wire Wire Line
-	4950 6300 4950 6200
-Wire Wire Line
 	1300 3000 1300 3100
 Wire Wire Line
@@
 Wire Wire Line
 	3450 2800 3450 2700
+Wire Wire Line
+	4950 6250 4950 6300
 $EndSCHEMATC

Commit message: Fix pins of FETs and other board tweaks.
Parts:
- removed Q1, Q2: 2N7002, TO_SOT_Packages_SMD:SOT-23_Handsoldering, symbol Q_NMOS_DGS
- removed Q3: BSS123, TO_SOT_Packages_SMD:SOT-23_Handsoldering, symbol Q_NMOS_DGS
- added Q1, Q2, Q3: 2N7002, TO_SOT_Packages_SMD:SOT-23_Handsoldering, symbol Q_NMOS_DGS-2N7002
- J6: footprint Connectors_Terminal_Blocks:TerminalBlock_Pheonix_MPT-2.54mm_3pol -> Connectors_Terminal_Blocks:TerminalBlock_Pheonix_MKDS1.5-3pol
Changed lines of the file:
@@
 F 0 "J6" H 10200 4150 50  0001 C TNN
 F 1 "Screw_Terminal_1x03" V 10050 3800 50  0000 C TNN
-F 2 "Connectors_Terminal_Blocks:TerminalBlock_Pheonix_MPT-2.54mm_3pol" H 10200 3475 50  0001 C CNN
+F 2 "Connectors_Terminal_Blocks:TerminalBlock_Pheonix_MKDS1.5-3pol" H 10200 3475 50  0001 C CNN
 F 3 "" H 10175 3900 50  0001 C CNN
 	1    10200 3800
@@
 $EndComp
 $Comp
-L Q_NMOS_DGS Q1
-U 1 1 5995F932
-P 1800 6950
-F 0 "Q1" H 2000 6950 50  0000 L CNN
-F 1 "2N7002" H 2000 6850 50  0000 L CNN
-F 2 "TO_SOT_Packages_SMD:SOT-23_Handsoldering" H 2000 7050 50  0001 C CNN
-F 3 "" H 1800 6950 50  0001 C CNN
-	1    1800 6950
-	1    0    0    -1
-$EndComp
-$Comp
 L GND #PWR037
 U 1 1 59960713
@@
 $EndComp
 $Comp
-L Q_NMOS_DGS Q2
-U 1 1 59960D3D
-P 3700 6950
-F 0 "Q2" H 3900 6950 50  0000 L CNN
-F 1 "2N7002" H 3900 6850 50  0000 L CNN
-F 2 "TO_SOT_Packages_SMD:SOT-23_Handsoldering" H 3900 7050 50  0001 C CNN
-F 3 "" H 3700 6950 50  0001 C CNN
-	1    3700 6950
-	1    0    0    -1
-$EndComp
-$Comp
 L GND #PWR040
 U 1 1 59960D47
@@
 F 3 "" H 6000 4100 50  0001 C CNN
 	1    6000 4100
-	1    0    0    -1
-$EndComp
-$Comp
-L Q_NMOS_DGS Q3
-U 1 1 59961F66
-P 6800 4100
-F 0 "Q3" H 7000 4100 50  0000 L CNN
-F 1 "BSS123" H 7000 4000 50  0000 L CNN
-F 2 "TO_SOT_Packages_SMD:SOT-23_Handsoldering" H 7000 4200 50  0001 C CNN
-F 3 "" H 6800 4100 50  0001 C CNN
-	1    6800 4100
 	1    0    0    -1
 $EndComp
@@
 Wire Wire Line
 	4950 6250 4950 6300
+$Comp
+L Q_NMOS_DGS-2N7002 Q1
+U 1 1 59C2466A
+P 1800 6950
+F 0 "Q1" H 2000 7000 50  0000 L CNN
+F 1 "2N7002" H 2000 6900 50  0000 L CNN
+F 2 "TO_SOT_Packages_SMD:SOT-23_Handsoldering" H 2000 7050 50  0001 C CNN
+F 3 "" H 1800 6950 50  0001 C CNN
+	1    1800 6950
+	1    0    0    -1
+$EndComp
+$Comp
+L Q_NMOS_DGS-2N7002 Q2
+U 1 1 59C2475D
+P 3700 6950
+F 0 "Q2" H 3900 7000 50  0000 L CNN
+F 1 "2N7002" H 3900 6900 50  0000 L CNN
+F 2 "TO_SOT_Packages_SMD:SOT-23_Handsoldering" H 3900 7050 50  0001 C CNN
+F 3 "" H 3700 6950 50  0001 C CNN
+	1    3700 6950
+	1    0    0    -1
+$EndComp
+$Comp
+L Q_NMOS_DGS-2N7002 Q3
+U 1 1 59C247E6
+P 6800 4100
+F 0 "Q3" H 7000 4150 50  0000 L CNN
+F 1 "2N7002" H 7000 4050 50  0000 L CNN
+F 2 "TO_SOT_Packages_SMD:SOT-23_Handsoldering" H 7000 4200 50  0001 C CNN
+F 3 "" H 6800 4100 50  0001 C CNN
+	1    6800 4100
+	1    0    0    -1
+$EndComp
 $EndSCHEMATC

Commit message: Final tweaks for version 2.
Connections:
- wire segments 98 -> 96
